File: pifire-relay-pwm-module-SSR.kicad_pcb (KiCad board)
At the start: 2 copper layers, 65 x 46 mm, 32 parts, among them J1 AC Terminal, J2 Relay Header, J3 PWM Fan Input, J5 Fan Header, K1 Power Relay, K2 Auger Relay, K3 Igniter Relay, Q1 BC547, Q2 BC547, Q3 BC547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

Commit message: Update to v1.0.1
Parts:
- R1, R10, R3, R7: value 4.7k -> 470
Other:
- board text added: "PiFire Relay PWM Module SSR v1.0.1"
- board text added: "v1.0.1 | December 2025 | Ben Parmeter"
- board text removed: "PiFire Relay PWM Module SSR v1.0.0"
- board text removed: "v1.0.0 | March 2024 | Ben Parmeter"
Changed lines of the file:
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@@
 			)
 		)
-		(property "Value" "4.7k"
+		(property "Value" "470"
 			(at 3.81 -2 0)
 			(layer "F.SilkS")
@@
 			)
 		)
-		(property "Value" "4.7k"
+		(property "Value" "470"
 			(at 4.37 -2.25 90)
 			(layer "F.SilkS")
@@
 			)
 		)
-		(property "Value" "4.7k"
+		(property "Value" "470"
 			(at 4.2275 -2.25 90)
 			(layer "F.SilkS")
@@
 			)
 		)
-		(property "Value" "4.7k"
+		(property "Value" "470"
 			(at 4.31 -2.25 90)
 			(layer "F.SilkS")
@@
 		)
 	)
-	(gr_text "v1.0.0 | March 2024 | Ben Parmeter"
+	(gr_text "v1.0.1 | December 2025 | Ben Parmeter"
 		(at 65 36.5 90)
 		(layer "B.SilkS")
@@
 			(justify left bottom mirror)
 		)
-		(render_cache "v1.0.0 | March 2024 | Ben Parmeter" 90
+		(render_cache "v1.0.1 | December 2025 | Ben Parmeter" 90
 			(polygon
 				(pts
@@
 		)
 	)
-	(gr_text "PiFire Relay PWM Module SSR v1.0.0"
+	(gr_text "PiFire Relay PWM Module SSR v1.0.1"
 		(at 31.75 27.25 0)
 		(layer "F.SilkS")
@@
 			(justify left bottom)
 		)
-		(render_cache "PiFire Relay PWM Module SSR v1.0.0" 0
+		(render_cache "PiFire Relay PWM Module SSR v1.0.1" 0
 			(polygon
 				(pts
