File: pifire-relay-pwm-module-SSR.kicad_sch (KiCad schematic)
At the start: 32 parts, among them J1 AC Terminal, J2 Relay Header, J3 PWM Fan Input, J5 Fan Header, K1 Power Relay, K2 Auger Relay, K3 Igniter Relay, Q1 BC547, Q2 BC547, Q3 BC547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

Commit message: Updated Schematic
Parts:
- R1, R10, R3, R7: value 4.7k -> 470
Changed lines of the file:
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@@
 (kicad_sch
-	(version 20231120)
+	(version 20250114)
 	(generator "eeschema")
-	(generator_version "8.0")
+	(generator_version "9.0")
 	(paper "A4")
 	(title_block
 		(title "PiFire Relay + PWM Fan Module")
-		(date "2024-03-11")
-		(rev "v1.0.0")
+		(date "2025-12-27")
+		(rev "v1.0.1")
 		(company "PiFire")
 		(comment 1 "https://github.com/nebhead/pifire")
 		(comment 2 "Ben Parmeter")
 	)
+	(rectangle
+		(start 17.78 90.17)
+		(end 101.6 163.83)
+		(stroke
+			(width 0)
+			(type default)
+		)
+		(fill
+			(type none)
+		)
+	)
+	(rectangle
+		(start 102.87 15.24)
+		(end 186.69 88.9)
+		(stroke
+			(width 0)
+			(type default)
+		)
+		(fill
+			(type none)
+		)
+	)
+	(rectangle
+		(start 17.78 15.24)
+		(end 101.6 88.9)
+		(stroke
+			(width 0)
+			(type default)
+		)
+		(fill
+			(type none)
+		)
+	)
+	(rectangle
+		(start 180.34 106.68)
+		(end 222.25 137.16)
+		(stroke
+			(width 0)
+			(type default)
+		)
+		(fill
+			(type none)
+		)
+	)
+	(rectangle
+		(start 118.11 91.44)
+		(end 166.37 129.54)
+		(stroke
+			(width 0)
+			(type default)
+		)
+		(fill
+			(type none)
+		)
+	)
+	(rectangle
+		(start 187.96 15.24)
+		(end 271.78 88.9)
+		(stroke
+			(width 0)
+			(type default)
+		)
+		(fill
+			(type none)
+		)
+	)
+	(rectangle
+		(start 121.92 142.24)
+		(end 166.37 162.56)
+		(stroke
+			(width 0)
+			(type default)
+		)
+		(fill
+			(type none)
+		)
+	)
+	(text "Fan Circuit"
+		(exclude_from_sim no)
+		(at 197.612 18.288 0)
+		(effects
+			(font
+				(size 1.27 1.27)
+			)
+		)
+	)
+	(text "Power Relay"
+		(exclude_from_sim no)
+		(at 25.654 93.726 0)
+		(effects
+			(font
+				(size 1.27 1.27)
+			)
+		)
+	)
+	(text "Fuses (F1-3): \n  Littelfuse 2A Slow Blow (39212000000)\n  https://www.digikey.com/en/products/detail/littelfuse-inc/39212000000/653505"
+		(exclude_from_sim no)
+		(at 17.78 176.784 0)
+		(effects
+			(font
+				(size 1.27 1.27)
+				(thickness 0.254)
+				(bold yes)
+			)
+			(justify left)
+		)
+	)
+	(text "AC Terminal Block"
+		(exclude_from_sim no)
+		(at 135.128 145.034 0)
+		(effects
+			(font
+				(size 1.27 1.27)
+			)
+		)
+	)
+	(text "Auger Relay"
+		(exclude_from_sim no)
+		(at 25.146 18.034 0)
+		(effects
+			(font
+				(size 1.27 1.27)
+			)
+		)
+	)
+	(text "Relay/Fan Board Header"
+		(exclude_from_sim no)
+		(at 153.67 94.742 0)
+		(effects
+			(font
+				(size 1.27 1.27)
+			)
+		)
+	)
+	(text "Relays (K1-3): \n  G3MB-202P  5V 2A SSR  \n  https://www.amazon.com/dp/B082F8C1LX"
+		(exclude_from_sim no)
+		(at 17.526 169.672 0)
+		(effects
+			(font
+				(size 1.27 1.27)
+				(thickness 0.254)
+				(bold yes)
+			)
+			(justify left)
+		)
+	)
+	(text "Mounting Holes"
+		(exclude_from_sim no)
+		(at 188.722 108.966 0)
+		(effects
+			(font
+				(size 1.27 1.27)
+			)
+		)
+	)
+	(text "Igniter Relay"
+		(exclude_from_sim no)
+		(at 110.49 18.288 0)
+		(effects
+			(font
+				(size 1.27 1.27)
+			)
+		)
+	)
 	(junction
 		(at 41.91 120.65)
@@
 		)
 	)
-	(rectangle
-		(start 17.78 90.17)
-		(end 101.6 163.83)
-		(stroke
-			(width 0)
-			(type default)
-		)
-		(fill
-			(type none)
-		)
-	)
-	(rectangle
-		(start 102.87 15.24)
-		(end 186.69 88.9)
-		(stroke
-			(width 0)
-			(type default)
-		)
-		(fill
-			(type none)
-		)
-	)
-	(rectangle
-		(start 17.78 15.24)
-		(end 101.6 88.9)
-		(stroke
-			(width 0)
-			(type default)
-		)
-		(fill
-			(type none)
-		)
-	)
-	(rectangle
-		(start 180.34 106.68)
-		(end 222.25 137.16)
-		(stroke
-			(width 0)
-			(type default)
-		)
-		(fill
-			(type none)
-		)
-	)
-	(rectangle
-		(start 118.11 91.44)
-		(end 166.37 129.54)
-		(stroke
-			(width 0)
-			(type default)
-		)
-		(fill
-			(type none)
-		)
-	)
-	(rectangle
-		(start 187.96 15.24)
-		(end 271.78 88.9)
-		(stroke
-			(width 0)
-			(type default)
-		)
-		(fill
-			(type none)
-		)
-	)
-	(rectangle
-		(start 121.92 142.24)
-		(end 166.37 162.56)
-		(stroke
-			(width 0)
-			(type default)
-		)
-		(fill
-			(type none)
-		)
-	)
 	(image
 		(at 278.13 173.99)
@@
 		)
 	)
-	(text "Fan Circuit"
-		(exclude_from_sim no)
-		(at 197.612 18.288 0)
-		(effects
-			(font
-				(size 1.27 1.27)
-			)
-		)
-	)
-	(text "Power Relay"
-		(exclude_from_sim no)
-		(at 25.654 93.726 0)
-		(effects
-			(font
-				(size 1.27 1.27)
-			)
-		)
-	)
-	(text "Fuses (F1-3): \n  Littelfuse 2A Slow Blow (39212000000)\n  https://www.digikey.com/en/products/detail/littelfuse-inc/39212000000/653505"
-		(exclude_from_sim no)
-		(at 17.78 176.784 0)
-		(effects
-			(font
-				(size 1.27 1.27)
-				(thickness 0.254)
-				(bold yes)
-			)
-			(justify left)
-		)
-	)
-	(text "AC Terminal Block"
-		(exclude_from_sim no)
-		(at 135.128 145.034 0)
-		(effects
-			(font
-				(size 1.27 1.27)
-			)
-		)
-	)
-	(text "Auger Relay"
-		(exclude_from_sim no)
-		(at 25.146 18.034 0)
-		(effects
-			(font
-				(size 1.27 1.27)
-			)
-		)
-	)
-	(text "Relay/Fan Board Header"
-		(exclude_from_sim no)
-		(at 153.67 94.742 0)
-		(effects
-			(font
-				(size 1.27 1.27)
-			)
-		)
-	)
-	(text "Relays (K1-3): \n  G3MB-202P  5V 2A SSR  \n  https://www.amazon.com/dp/B082F8C1LX"
-		(exclude_from_sim no)
-		(at 17.526 169.672 0)
-		(effects
-			(font
-				(size 1.27 1.27)
-				(thickness 0.254)
-				(bold yes)
-			)
-			(justify left)
-		)
-	)
-	(text "Mounting Holes"
-		(exclude_from_sim no)
-		(at 188.722 108.966 0)
-		(effects
-			(font
-				(size 1.27 1.27)
-			)
-		)
-	)
-	(text "Igniter Relay"
-		(exclude_from_sim no)
-		(at 110.49 18.288 0)
-		(effects
-			(font
-				(size 1.27 1.27)
-			)
-		)
-	)
 	(global_label "+12V"
 		(shape input)
@@
 			)
 		)
-		(property "Value" "4.7k"
+		(property "Value" "470"
 			(at 34.29 116.84 90)
 			(effects
@@
 			)
 		)
-		(property "Value" "4.7k"
+		(property "Value" "470"
 			(at 119.38 46.99 90)
 			(effects
@@
 			)
 		)
-		(property "Value" "4.7k"
+		(property "Value" "470"
 			(at 217.17 73.66 90)
 			(effects
@@
 			)
 		)
-		(property "Value" "4.7k"
+		(property "Value" "470"
 			(at 35.56 46.99 90)
 			(effects
@@
 		)
 	)
+	(embedded_fonts no)
 )
